Commit message: Pointed the camera up a bit so that the wheel arches are not visible.

File: urdf/traethlin.urdf.xacro (robot description, xacro)
@@ -178,5 +178,5 @@
   </joint>
   <joint name="camera_base_joint" type="fixed">
-    <origin xyz="0.035 0 0.37" rpy="0 0.40 0"/>
+    <origin xyz="0.035 0 0.37" rpy="0 0.36 0"/>
     <parent link="cam_mount_link"/>
     <child link="camera_base"/>

Commit message: Can now use a realsense d455 or oak-d-s2 camera.

File: urdf/traethlin.urdf.xacro (robot description, xacro)
@@ -11,4 +11,6 @@
 -->
 <robot name="traethlin" xmlns:xacro="http://www.ros.org/wiki/xacro">
+  <xacro:arg name="camera_type" default="oak-d-s2" />
+  <!-- Possible values are 'oak-d-s2' or 'd455' -->
   <xacro:include filename="$(find traethlin_description)/urdf/traethlin_constants.xacro" />
   <xacro:include filename="$(find traethlin_description)/urdf/traethlin_shock_absorbers.xacro" />
@@ -203,13 +205,43 @@
     <child link="cam_mount_link"/>
   </joint>
-  <joint name="camera_base_joint" type="fixed">
-    <origin xyz="0.035 0 0.355" rpy="0 0.36 0"/>
-    <parent link="cam_mount_link"/>
-    <child link="camera_base"/>
-  </joint>
-  <!-- Camera -->
-  <link name="camera_base">
-    <xacro:null_inertial/>
-  </link>
+  <xacro:property name="cmp_camera_type" value="$(arg camera_type)"/>
+  <!-- realsense d455 camera -->
+  <xacro:if value="${cmp_camera_type == 'd455'}">
+    <link name="camera_base">
+      <xacro:null_inertial/>
+    </link>
+    <xacro:arg name="use_nominal_extrinsics" default="true"/>
+    <xacro:include
+      filename="$(find realsense2_description)/urdf/_d455.urdf.xacro" />
+    <xacro:sensor_d455 parent="camera_base"
+                       use_nominal_extrinsics="$(arg use_nominal_extrinsics)">
+      <origin xyz="0 0 0" rpy="0 0 0"/>
+    </xacro:sensor_d455>
+    <joint name="camera_base_joint" type="fixed">
+      <origin xyz="0.03 0 0.358" rpy="0 0.36 0"/>
+      <parent link="cam_mount_link"/>
+      <child link="camera_base"/>
+    </joint>
+  </xacro:if>
+  <!-- oak-d camera -->
+  <xacro:if value="${cmp_camera_type == 'oak-d-s2'}">
+    <xacro:arg name="camera_name"   default="camera" />
+    <xacro:arg name="camera_model"  default="OAK-D-S2" />
+    <xacro:arg name="base_frame"    default="oak-d_frame" />
+    <xacro:arg name="parent_frame"  default="camera_base" />
+    <xacro:arg name="cam_pos_x"     default="0.0" />
+    <xacro:arg name="cam_pos_y"     default="0.0" />
+    <xacro:arg name="cam_pos_z"     default="0.0" />
+    <xacro:arg name="cam_roll"      default="0.0" />
+    <xacro:arg name="cam_pitch"     default="0.0" />
+    <xacro:arg name="cam_yaw"       default="0.0" />
+    <xacro:include
+        filename="$(find depthai_descriptions)/urdf/depthai_descr.urdf.xacro"/>
+    <joint name="camera_base_joint" type="fixed">
+      <origin xyz="0.048 0 0.365" rpy="0 0.36 0"/>
+      <parent link="cam_mount_link"/>
+      <child link="camera_base"/>
+    </joint>
+  </xacro:if>
   <joint name="thermal_joint" type="fixed">
     <origin xyz="0.18 0 0.06" rpy="0 0.1 0"/>
@@ -255,9 +287,4 @@
                     wheel_mass="${rear_wheel_mass}"
                     axle_eff_limit="${rear_axle_eff_limit}"/>
-  <xacro:arg name="use_nominal_extrinsics" default="true"/>
-  <xacro:include filename="$(find realsense2_description)/urdf/_d455.urdf.xacro" />
-  <xacro:sensor_d455 parent="camera_base" use_nominal_extrinsics="$(arg use_nominal_extrinsics)">
-    <origin xyz="0 0 0" rpy="0 0 0"/>
-  </xacro:sensor_d455>
   <gazebo>
     <plugin name="gazebo_ros_ackermann_drive"

Commit message: Better dealing with stl file access.

File: urdf/traethlin.urdf.xacro (robot description, xacro)
@@ -100,5 +100,5 @@
               rpy="0 0 0"/>
       <geometry>
-        <mesh filename="file://$(find traethlin_description)/meshes/chassis.stl" scale="0.001 0.001 0.001" />
+        <mesh filename="package://traethlin_description/meshes/chassis.stl" scale="0.001 0.001 0.001" />
       </geometry>
       <material name="chassis_mat"/>
@@ -111,5 +111,5 @@
               <!-- rpy="0 0 0"/> -->
       <geometry>
-        <mesh filename="file://$(find traethlin_description)/meshes/chassis.stl" scale="0.001 0.001 0.001" />
+        <mesh filename="package://traethlin_description/meshes/chassis.stl" scale="0.001 0.001 0.001" />
       </geometry>
     </collision>
@@ -185,5 +185,5 @@
       <origin xyz="0 0 0" rpy="0 0 0"/>
       <geometry>
-        <mesh filename="file://$(find traethlin_description)/meshes/camera_assembly.stl" scale="0.001 0.001 0.001" />
+        <mesh filename="package://traethlin_description/meshes/camera_assembly.stl" scale="0.001 0.001 0.001" />
       </geometry>
       <material name="orange"/>
@@ -192,5 +192,5 @@
       <origin xyz="0 0 0" rpy="0 0 0"/>
       <geometry>
-        <mesh filename="file://$(find traethlin_description)/meshes/camera_assembly.stl" scale="0.001 0.001 0.001" />
+        <mesh filename="package://traethlin_description/meshes/camera_assembly.stl" scale="0.001 0.001 0.001" />
       </geometry>
     </collision>
@@ -226,7 +226,7 @@
   <!-- oak-d camera -->
   <xacro:if value="${cmp_camera_type == 'oak-d-s2'}">
-    <xacro:arg name="camera_name"   default="camera" />
+    <xacro:arg name="camera_name"   default="oak" />
     <xacro:arg name="camera_model"  default="OAK-D-S2" />
-    <xacro:arg name="base_frame"    default="oak-d_frame" />
+    <!--    <xacro:arg name="base_frame"    default="oak-d_frame" />-->
     <xacro:arg name="parent_frame"  default="camera_base" />
     <xacro:arg name="cam_pos_x"     default="0.0" />

Commit message: Fixed inertia of wheels.

File: urdf/traethlin.urdf.xacro (robot description, xacro)
@@ -45,8 +45,7 @@
        MOI is calculated from platform calibration data using bifilar pendulum
        method
-       TODO: remove inner_rad
       -->
-  <xacro:macro name="thick_walled_tube_inertial"
-               params="inner_rad outer_rad height mass">
+  <xacro:macro name="cylinder_inertial"
+               params="outer_rad height mass">
     <inertial>
       <mass value="${mass}"/>
@@ -57,14 +56,7 @@
         iyz = "0"
         izz="${(mass*outer_rad*outer_rad)/2}"/>
-      <!--ixx="${(1 / 12) * mass * (3 * (inner_rad * inner_rad +
-                    outer_rad * outer_rad) + height * height)}"
-               ixy="0" ixz="0"
-               iyy="0.0224048079"
-               iyz="0"
-               izz="${mass * (inner_rad * inner_rad +
-                    outer_rad * outer_rad) / 2}"-->
     </inertial>
   </xacro:macro>
-  <xacro:macro  name="thick_walled_tube_inertial"
+<!--  <xacro:macro  name="thick_walled_tube_inertial"
                 params="inner_rad outer_rad height mass">
     <inertial>
@@ -77,5 +69,5 @@
         izz="${mass*outer_rad/2}"/>
       </inertial>
-  </xacro:macro>
+  </xacro:macro>-->
   <xacro:macro name="solid_cube_inertial"
                params="x y z mass">

File: urdf/traethlin_wheels.xacro (robot description, xacro)
@@ -79,6 +79,6 @@
         </geometry>
       </collision>-->
-      <xacro:thick_walled_tube_inertial
-          inner_rad="${hub_dia / 2.0}" outer_rad="${tire_dia / 2.0}"
+      <xacro:cylinder_inertial
+          outer_rad="${tire_dia / 2.0}"
           height="${tire_width}" mass="${wheel_mass}"/>
     </link>

Commit message: Maybe better null inertia.

File: urdf/traethlin.urdf.xacro (robot description, xacro)
@@ -36,6 +36,8 @@
   <xacro:macro name="null_inertial">
     <inertial>
-      <mass value="8e-3"/>
-      <inertia ixx="8e-3" ixy="0" ixz="0" iyy="8e-3" iyz="0" izz="8e-3"/>
+      <!-- <mass value="8e-3"/>
+      <inertia ixx="8e-3" ixy="0" ixz="0" iyy="8e-3" iyz="0" izz="8e-3"/> -->
+      <mass value="0.05"/>
+      <inertia ixx="0.0005" ixy="0" ixz="0" iyy="0.0005" iyz="0" izz="0.0005"/>
     </inertial>
   </xacro:macro>
@@ -52,5 +54,6 @@
       <inertia
         ixx="${(mass*(3*outer_rad*outer_rad+height*height))/12}"
-        ixy = "0" ixz = "0"
+        ixy = "0"
+        ixz = "0"
         iyy="${(mass*(3*outer_rad*outer_rad+height*height))/12}"
         iyz = "0"
@@ -58,16 +61,17 @@
     </inertial>
   </xacro:macro>
-<!--  <xacro:macro  name="thick_walled_tube_inertial"
-                params="inner_rad outer_rad height mass">
+  <!-- <xacro:macro  name="cylinder_inertial"
+                params="outer_rad height mass">
     <inertial>
       <mass value="${mass}"/>
       <inertia
         ixx="${(mass*(3*outer_rad*outer_rad+height*height))/12}"
-        ixy = "0" ixz = "0"
+        ixy = "0"
+        ixz = "0"
         iyy="${(mass*(3*outer_rad*outer_rad+height*height))/12}"
         iyz = "0"
         izz="${mass*outer_rad/2}"/>
       </inertial>
-  </xacro:macro>-->
+  </xacro:macro> -->
   <xacro:macro name="solid_cube_inertial"
                params="x y z mass">
@@ -75,5 +79,6 @@
       <mass value="${mass}"/>
       <inertia ixx="${mass*(y*y+z*z)/12}"
-        ixy = "0" ixz = "0"
+        ixy = "0"
+        ixz = "0"
         iyy="${mass*(x*x+z*z)/12}"
         iyz = "0"
@@ -312,6 +317,6 @@
       <linear_velocity_i_range>0 0</linear_velocity_i_range>
       <!-- output -->
-      <publish_odom>false</publish_odom>
-      <publish_odom_tf>false</publish_odom_tf>
+      <publish_odom>true</publish_odom>
+      <publish_odom_tf>true</publish_odom_tf>
       <publish_wheel_tf>true</publish_wheel_tf>
       <publish_distance>true</publish_distance>

Commit message: Fixed inertia issue that resulted in exploding robot.

File: urdf/traethlin.urdf.xacro (robot description, xacro)
@@ -38,28 +38,13 @@
       <!-- <mass value="8e-3"/>
       <inertia ixx="8e-3" ixy="0" ixz="0" iyy="8e-3" iyz="0" izz="8e-3"/> -->
-      <mass value="0.05"/>
-      <inertia ixx="0.0005" ixy="0" ixz="0" iyy="0.0005" iyz="0" izz="0.0005"/>
+      <mass value="0.005"/>
+      <inertia ixx="0.001" ixy="0" ixz="0" iyy="0.001" iyz="0" izz="0.001"/>
     </inertial>
   </xacro:macro>
-  <!-- Inertia of a thick-walled cylindrical tube with open ends. Height is
-       measured along the z axis, which is the tube's axis. inner_rad and
-       outer_rad are the tube's inner and outer radii, respectively. Pitch
-       MOI is calculated from platform calibration data using bifilar pendulum
-       method
+  <!-- Inertia of a cylinder. Height is
+       measured along the z axis, which is the cylinder's axis.
+       outer_rad is the cylinder's outer radius.
       -->
-  <xacro:macro name="cylinder_inertial"
-               params="outer_rad height mass">
-    <inertial>
-      <mass value="${mass}"/>
-      <inertia
-        ixx="${(mass*(3*outer_rad*outer_rad+height*height))/12}"
-        ixy = "0"
-        ixz = "0"
-        iyy="${(mass*(3*outer_rad*outer_rad+height*height))/12}"
-        iyz = "0"
-        izz="${(mass*outer_rad*outer_rad)/2}"/>
-    </inertial>
-  </xacro:macro>
-  <!-- <xacro:macro  name="cylinder_inertial"
+  <xacro:macro  name="cylinder_inertial"
                 params="outer_rad height mass">
     <inertial>
@@ -67,11 +52,10 @@
       <inertia
         ixx="${(mass*(3*outer_rad*outer_rad+height*height))/12}"
-        ixy = "0"
-        ixz = "0"
+        ixy = "0" ixz = "0"
         iyy="${(mass*(3*outer_rad*outer_rad+height*height))/12}"
         iyz = "0"
         izz="${mass*outer_rad/2}"/>
       </inertial>
-  </xacro:macro> -->
+  </xacro:macro>
   <xacro:macro name="solid_cube_inertial"
                params="x y z mass">
@@ -79,6 +63,5 @@
       <mass value="${mass}"/>
       <inertia ixx="${mass*(y*y+z*z)/12}"
-        ixy = "0"
-        ixz = "0"
+        ixy = "0" ixz = "0"
         iyy="${mass*(x*x+z*z)/12}"
         iyz = "0"
@@ -317,6 +300,6 @@
       <linear_velocity_i_range>0 0</linear_velocity_i_range>
       <!-- output -->
-      <publish_odom>true</publish_odom>
-      <publish_odom_tf>true</publish_odom_tf>
+      <publish_odom>false</publish_odom>
+      <publish_odom_tf>false</publish_odom_tf>
       <publish_wheel_tf>true</publish_wheel_tf>
       <publish_distance>true</publish_distance>

Commit message: Tilted camera up a bit to avoid the thermal camera.

File: urdf/traethlin.urdf.xacro (robot description, xacro)
@@ -219,5 +219,5 @@
         filename="$(find depthai_descriptions)/urdf/depthai_descr.urdf.xacro"/>
     <joint name="camera_base_joint" type="fixed">
-      <origin xyz="0.048 0 0.365" rpy="0 0.36 0"/>
+      <origin xyz="0.048 0 0.365" rpy="0 0.335 0"/>
       <parent link="cam_mount_link"/>
       <child link="camera_base"/>

Commit message: Changed tilt of oak camera to align the PC better.

File: urdf/traethlin.urdf.xacro (robot description, xacro)
@@ -219,5 +219,5 @@
         filename="$(find depthai_descriptions)/urdf/depthai_descr.urdf.xacro"/>
     <joint name="camera_base_joint" type="fixed">
-      <origin xyz="0.048 0 0.365" rpy="0 0.335 0"/>
+      <origin xyz="0.048 0 0.365" rpy="0 0.4 0"/>
       <parent link="cam_mount_link"/>
       <child link="camera_base"/>

Commit message: Fixed inertia error for wheels.

File: urdf/traethlin.urdf.xacro (robot description, xacro)
@@ -55,5 +55,5 @@
         iyy="${(mass*(3*outer_rad*outer_rad+height*height))/12}"
         iyz = "0"
-        izz="${mass*outer_rad/2}"/>
+        izz="${mass*outer_rad*outer_rad/2}"/>
       </inertial>
   </xacro:macro>

File: urdf/traethlin_wheels.xacro (robot description, xacro)
@@ -73,12 +73,6 @@
         </geometry>
       </collision>
-      <!--<collision name="collision">
-        <origin xyz="0 0 0"/>
-        <geometry>
-          <mesh filename="${wheel_model}" scale="0.632 0.632 0.661"/>
-        </geometry>
-      </collision>-->
       <xacro:cylinder_inertial
-          outer_rad="${tire_dia / 2.0}"
+          outer_rad="${tire_dia/2}"
           height="${tire_width}" mass="${wheel_mass}"/>
     </link>

Commit message: Spelling of tyre.

File: urdf/traethlin.urdf.xacro (robot description, xacro)
@@ -249,20 +249,20 @@
   <xacro:front_wheel lr_prefix="left" fr_prefix="front"
                      lr_reflect="1" fr_reflect="1"
-                     tire_width="${front_tire_width}"
+                     tyre_width="${front_tyre_width}"
                      wheel_mass="${front_wheel_mass}"
                      axle_eff_limit="${front_axle_eff_limit}"/>
   <xacro:front_wheel lr_prefix="right" fr_prefix="front"
                      lr_reflect="-1" fr_reflect="1"
-                     tire_width="${front_tire_width}"
+                     tyre_width="${front_tyre_width}"
                      wheel_mass="${front_wheel_mass}"
                      axle_eff_limit="${front_axle_eff_limit}"/>
   <xacro:rear_wheel lr_prefix="left" fr_prefix="rear"
                     lr_reflect="1" fr_reflect="-1"
-                    tire_width="${rear_tire_width}"
+                    tyre_width="${rear_tyre_width}"
                     wheel_mass="${rear_wheel_mass}"
                     axle_eff_limit="${rear_axle_eff_limit}"/>
   <xacro:rear_wheel lr_prefix="right" fr_prefix="rear"
                     lr_reflect="-1" fr_reflect="-1"
-                    tire_width="${rear_tire_width}"
+                    tyre_width="${rear_tyre_width}"
                     wheel_mass="${rear_wheel_mass}"
                     axle_eff_limit="${rear_axle_eff_limit}"/>

File: urdf/traethlin_constants.xacro (robot description, xacro)
@@ -34,21 +34,21 @@
   <xacro:property name="chassis_cm_to_rear_shock" value="0.155"/>
   <xacro:property name="chassis_cm_to_front_shock" value="0.155"/>
-  <!-- hub_dia and tire_dia are the diameters of the hub and tire,
+  <!-- hub_dia and tyre_dia are the diameters of the hub and tyre,
        respectively. hex_hub_depth is the distance that the hex hub is
-       inset from the outer edge of the tire. It is set so that each wheel
-       is a "zero offset" wheel. hex_hub_depth = tire_width / 2 -
+       inset from the outer edge of the tyre. It is set so that each wheel
+       is a "zero offset" wheel. hex_hub_depth = tyre_width / 2 -
        axle_length. -->
   <!--<xacro:property name="hub_dia" value="0.024"/>
-  <xacro:property name="tire_dia" value="0.19"/>
-  <xacro:property name="front_tire_width" value="0.072644"/>
+  <xacro:property name="tyre_dia" value="0.19"/>
+  <xacro:property name="front_tyre_width" value="0.072644"/>
   <xacro:property name="front_wheel_mass" value="0.82"/>
-  <xacro:property name="rear_tire_width" value="0.0762"/>
+  <xacro:property name="rear_tyre_width" value="0.0762"/>
   <xacro:property name="rear_wheel_mass" value="0.89"/>-->
   <xacro:property name="hub_dia" value="0.015"/>
-  <xacro:property name="tire_dia" value="0.110"/>
+  <xacro:property name="tyre_dia" value="0.110"/>
   <!-- <xacro:property name="hex_hub_depth" value="0.0"/>  -->
-  <xacro:property name="front_tire_width" value="0.07"/>
+  <xacro:property name="front_tyre_width" value="0.07"/>
   <xacro:property name="front_wheel_mass" value="0.115"/><!--0.115-->
-  <xacro:property name="rear_tire_width" value="0.07"/>
+  <xacro:property name="rear_tyre_width" value="0.07"/>
   <xacro:property name="rear_wheel_mass" value="0.115"/>
   <!-- hex_hub_dist is the distance between left and right hex hubs when
@@ -97,5 +97,5 @@
          5.12766 N m
        max_speed = 60mph = 26.82 m/s
-       axle_vel_limit = (2 * pi) * (max_speed / (pi * tire_dia)) =
+       axle_vel_limit = (2 * pi) * (max_speed / (pi * tyre_dia)) =
           2*26.82/0.19 = 282.315789474 rad/s
        -->

File: urdf/traethlin_wheels.xacro (robot description, xacro)
@@ -12,5 +12,5 @@
 <robot name="traethlin" xmlns:xacro="http://www.ros.org/wiki/xacro">
   <!-- The "wheel" macro defines an axle carrier, axle, and wheel. -->
-  <xacro:macro name="wheel" params="lr_prefix fr_prefix lr_reflect tire_width wheel_mass axle_eff_limit wheel_model cant">
+  <xacro:macro name="wheel" params="lr_prefix fr_prefix lr_reflect tyre_width wheel_mass axle_eff_limit wheel_model cant">
     <link name="${lr_prefix}_${fr_prefix}_axle_carrier">
       <xacro:null_inertial/>
@@ -63,5 +63,5 @@
 -->
         <geometry>
-          <cylinder radius="${tire_dia/2}" length="${tire_width}"/>
+          <cylinder radius="${tyre_dia/2}" length="${tyre_width}"/>
         </geometry>
         <material name="black"/>
@@ -70,10 +70,10 @@
         <origin xyz="0 0 0" rpy="0 0 0"/>
         <geometry>
-          <cylinder radius="${tire_dia/2}" length="${tire_width}"/>
+          <cylinder radius="${tyre_dia/2}" length="${tyre_width}"/>
         </geometry>
       </collision>
       <xacro:cylinder_inertial
-          outer_rad="${tire_dia/2}"
-          height="${tire_width}" mass="${wheel_mass}"/>
+          outer_rad="${tyre_dia/2}"
+          height="${tyre_width}" mass="${wheel_mass}"/>
     </link>
     <gazebo reference="${lr_prefix}_${fr_prefix}_wheel">
@@ -96,5 +96,5 @@
   <!-- Front wheel -->
   <xacro:macro name="front_wheel"
-               params="lr_prefix fr_prefix lr_reflect fr_reflect tire_width
+               params="lr_prefix fr_prefix lr_reflect fr_reflect tyre_width
                        wheel_mass axle_eff_limit">
     <xacro:front_shock lr_prefix="${lr_prefix}" fr_prefix="${fr_prefix}"
@@ -126,5 +126,5 @@
     </transmission>
     <xacro:wheel lr_prefix="${lr_prefix}" fr_prefix="${fr_prefix}"
-                 lr_reflect="${lr_reflect}" tire_width="${tire_width}"
+                 lr_reflect="${lr_reflect}" tyre_width="${tyre_width}"
                  wheel_mass="${wheel_mass}"
                  axle_eff_limit="${axle_eff_limit}"
@@ -134,5 +134,5 @@
   <!-- Rear wheel -->
   <xacro:macro name="rear_wheel"
-               params="lr_prefix fr_prefix lr_reflect fr_reflect tire_width
+               params="lr_prefix fr_prefix lr_reflect fr_reflect tyre_width
                        wheel_mass axle_eff_limit">
     <xacro:rear_shock lr_prefix="${lr_prefix}" fr_prefix="${fr_prefix}"
@@ -140,5 +140,5 @@
                  child="${lr_prefix}_${fr_prefix}_axle_carrier"/>
     <xacro:wheel lr_prefix="${lr_prefix}" fr_prefix="${fr_prefix}"
-                 lr_reflect="${lr_reflect}" tire_width="${tire_width}"
+                 lr_reflect="${lr_reflect}" tyre_width="${tyre_width}"
                  wheel_mass="${wheel_mass}"
                  axle_eff_limit="${axle_eff_limit}"

Commit message: Adjusted angle of the camera.

File: urdf/traethlin.urdf.xacro (robot description, xacro)
@@ -199,5 +199,5 @@
     </xacro:sensor_d455>
     <joint name="camera_base_joint" type="fixed">
-      <origin xyz="0.05 0 0.39" rpy="0 0.36 0"/>
+      <origin xyz="0.05 0 0.39" rpy="0 0.38 0"/>
       <parent link="cam_mount_link"/>
       <child link="camera_base"/>
@@ -219,5 +219,5 @@
         filename="$(find depthai_descriptions)/urdf/depthai_descr.urdf.xacro"/>
     <joint name="camera_base_joint" type="fixed">
-      <origin xyz="0.048 0 0.365" rpy="0 0.4 0"/>
+      <origin xyz="0.05 0 0.39" rpy="0 0.38 0"/>
       <parent link="cam_mount_link"/>
       <child link="camera_base"/>

Commit message: New mdel for the camera mast.

File: urdf/traethlin.urdf.xacro (robot description, xacro)
@@ -130,5 +130,5 @@
   </link>
   <joint name="box_of_goodies_to_chassis_joint" type="fixed">
-    <origin xyz="-0.105 0 0.115" rpy="0 0 0"/>
+    <origin xyz="-0.103 0 0.114" rpy="0 0 0"/>
     <parent link="chassis_link"/>
     <child link="box_of_goodies_link"/>
@@ -183,5 +183,5 @@
   </gazebo>
   <joint name="cam_mount_joint" type="fixed">
-    <origin xyz="-0.206 0 0.025" rpy="0 0 0"/>
+    <origin xyz="-0.206 0 0.037" rpy="0 0 0"/>
     <parent link="chassis_link"/>
     <child link="cam_mount_link"/>
@@ -221,5 +221,5 @@
         filename="$(find depthai_descriptions)/urdf/depthai_descr.urdf.xacro"/>
     <joint name="camera_base_joint" type="fixed">
-      <origin xyz="0.05 0 0.39" rpy="0 0.38 0"/>
+      <origin xyz="0.053 0 0.372" rpy="0 0.38 0"/>
       <parent link="cam_mount_link"/>
       <child link="camera_base"/>
