Commit message: Tweaked camera pose for the current setup.

File: urdf/traethlin.urdf.xacro (robot description, xacro)
@@ -201,5 +201,5 @@
     </xacro:sensor_d455>
     <joint name="camera_base_joint" type="fixed">
-      <origin xyz="0.05 0 0.39" rpy="0 0.38 0"/>
+      <origin xyz="0.05 0 0.368" rpy="0 0.28 0"/>
       <parent link="cam_mount_link"/>
       <child link="camera_base"/>
@@ -221,5 +221,5 @@
         filename="$(find depthai_descriptions)/urdf/depthai_descr.urdf.xacro"/>
     <joint name="camera_base_joint" type="fixed">
-      <origin xyz="0.053 0 0.372" rpy="0 0.38 0"/>
+      <origin xyz="0.053 0 0.368" rpy="0 0.28 0"/>
       <parent link="cam_mount_link"/>
       <child link="camera_base"/>
