Commit message: Added some colours.

File: urdf/traethlin.gazebo.xacro (robot description, xacro)
@@ -129,4 +129,5 @@
   </gazebo>
   <gazebo reference="thermal_link">
+    <material>Gazebo/White</material>
     <sensor type="camera" name="thermal_camera">
       <camera name="thermal_camera">
@@ -150,4 +151,5 @@
     </sensor>
   </gazebo>
+  <!--
   <gazebo reference="lidar">
     <sensor name="sensor_ray" type="ray">
@@ -178,3 +180,4 @@
     </sensor>
   </gazebo>
+  -->
 </robot>

File: urdf/traethlin.urdf.xacro (robot description, xacro)
@@ -15,4 +15,7 @@
   <xacro:include filename="$(find traethlin_description)/urdf/traethlin_wheels.xacro" />
   <xacro:include filename="$(find traethlin_description)/urdf/traethlin.gazebo.xacro" />
+  <material name="black">
+    <color rgba="0.0 0.0 0.0 1"/>
+  </material>
   <material name="chassis_mat">
     <color rgba="0.2 0.2 0.2 1"/>
@@ -20,4 +23,10 @@
   <material name="lightgrey">
     <color rgba="0.8 0.8 0.8 1"/>
+  </material>
+  <material name="orange">
+    <color rgba="1.0 0.5 0.05 1"/>
+  </material>
+  <material name="off_white">
+    <color rgba="0.9 0.9 0.5 1"/>
   </material>
   <!-- Null inertial element. This is needed to make the model work with
@@ -78,13 +87,5 @@
     </inertial>
   </xacro:macro>
-  <!-- base_link must have geometry so that its axes can be displayed in
-       rviz. -->
   <link name="base_link">
-<!--    <visual>
-      <geometry>
-        <box size="0.01 0.01 0.01"/>
-      </geometry>
-      <material name="chassis_mat"/>
-    </visual>-->
   </link>
   <gazebo reference="base_link">
@@ -94,6 +95,4 @@
   <link name="chassis_link">
     <visual>
-      <!--<origin xyz="${-chassis_length/2 + 0.15} 0 ${-chassis_cm_height}"
-              rpy="0 0 0"/>-->
       <origin xyz="${chassis_length_offset} 0 ${chassis_vertical_offset}"
               rpy="0 0 0"/>
@@ -120,4 +119,5 @@
   </link>
   <gazebo reference="chassis_link">
+    <material>Gazebo/DarkGrey</material>
     <mu1>0.2</mu1>
     <mu2>0.2</mu2>
@@ -162,5 +162,5 @@
         <mesh filename="file://$(find traethlin_description)/meshes/camera_assembly.stl" scale="0.001 0.001 0.001" />
       </geometry>
-      <material name="lightgrey"/>
+      <material name="orange"/>
     </visual>
     <collision>
@@ -172,4 +172,7 @@
     <xacro:null_inertial/>
   </link>
+  <gazebo reference="cam_mount_link">
+    <material>Gazebo/Orange</material>
+  </gazebo>
   <joint name="cam_mount_joint" type="fixed">
     <origin xyz="-0.19 0 0.04" rpy="0 0 0"/>
@@ -184,22 +187,8 @@
   <!-- Camera -->
   <link name="camera_base">
-    <!--<collision>
-      <origin xyz="0 0 0" rpy="0 0 0"/>
-      <geometry>
-    <box size="0.03 0.12 0.03"/>
-      </geometry>
-      <material name="lightgrey"/>
-    </collision>
-    <visual>
-      <origin xyz="0 0 0" rpy="0 0 0"/>
-      <geometry>
-        <box size="0.03 0.12 0.03"/>
-      </geometry>
-      <material name="lightgrey"/>
-    </visual>-->
     <xacro:null_inertial/>
   </link>
   <joint name="thermal_joint" type="fixed">
-    <origin xyz="0.20 0 0.07" rpy="0 0 0"/>
+    <origin xyz="0.18 0 0.06" rpy="0 0.1 0"/>
     <parent link="chassis_link"/>
     <child link="thermal_link"/>
@@ -207,18 +196,17 @@
   <!-- Thermal Camera -->
   <link name="thermal_link">
-    <!--<collision>
-      <origin xyz="0 0 0" rpy="0 0 0"/>
-      <geometry>
-    <box size="0.03 0.12 0.03"/>
-      </geometry>
-      <material name="lightgrey"/>
+    <collision>
+      <origin xyz="0 0 0" rpy="0 0 0"/>
+      <geometry>
+        <box size="0.01 0.04 0.04"/>
+      </geometry>
     </collision>
     <visual>
       <origin xyz="0 0 0" rpy="0 0 0"/>
       <geometry>
-        <box size="0.03 0.12 0.03"/>
-      </geometry>
-      <material name="lightgrey"/>
-    </visual>-->
+        <box size="0.01 0.04 0.04"/>
+      </geometry>
+      <material name="off_white"/>
+    </visual>
     <xacro:null_inertial/>
   </link>

File: urdf/traethlin_wheels.xacro (robot description, xacro)
@@ -63,4 +63,5 @@
           <cylinder radius="${tire_dia/2}" length="${rear_tire_width*0.1}"/>
         </geometry> -->
+        <material name="black"/>
       </visual>
       <!--<collision name="collision">
@@ -88,4 +89,5 @@
     </link>
     <gazebo reference="${lr_prefix}_${fr_prefix}_wheel">
+      <material>Gazebo/Black</material>
       <mu1>10</mu1>
       <mu2>10</mu2>

Commit message: Added box of goodies.

File: urdf/traethlin.gazebo.xacro (robot description, xacro)
@@ -43,4 +43,5 @@
   </gazebo>
   <gazebo reference="gps_link">
+    <material>Gazebo/Black</material>
     <sensor name="gps" type="gps">
       <always_on>true</always_on>

File: urdf/traethlin.urdf.xacro (robot description, xacro)
@@ -128,11 +128,27 @@
     <child link="chassis_link"/>
   </joint>
+  <!-- Box of goodies! -->
+  <link name="box_of_goodies_link">
+    <visual>
+      <origin xyz="0 0 0" rpy="0 0 0"/>
+      <geometry>
+        <box size="0.15 0.15 0.07"/>
+      </geometry>
+      <material name="lightgrey"/>
+    </visual>
+    <collision>
+      <origin xyz="0 0 0" rpy="0 0 0"/>
+      <geometry>
+        <box size="0.15 0.15 0.07"/>
+      </geometry>
+    </collision>
+    <xacro:null_inertial/>
+  </link>
+  <joint name="box_of_goodies_to_chassis_joint" type="fixed">
+    <origin xyz="-0.10 0 0.10" rpy="0 0 0"/>
+    <parent link="chassis_link"/>
+    <child link="box_of_goodies_link"/>
+  </joint>
   <link name="imu_link">
-    <collision>
-      <origin xyz="0 0 0" rpy="0 0 0"/>
-      <geometry>
-        <box size="0.01 0.01 0.01"/>
-      </geometry>
-    </collision>
     <xacro:null_inertial/>
   </link>
@@ -146,7 +162,14 @@
       <origin xyz="0 0 0" rpy="0 0 0"/>
       <geometry>
-        <box size="0.01 0.01 0.01"/>
-      </geometry>
-    </collision>
+        <cylinder radius="0.015" length="0.01"/>
+      </geometry>
+    </collision>
+    <visual>
+      <origin xyz="0 0 0" rpy="0 0 0"/>
+      <geometry>
+        <cylinder radius="0.015" length="0.01"/>
+      </geometry>
+      <material name="black"/>
+    </visual>
     <xacro:null_inertial/>
   </link>
@@ -211,58 +234,4 @@
     <xacro:null_inertial/>
   </link>
-<!--
-  <joint name="side_camera_joint" type="fixed">
-    <axis xyz="0 1 0" />
-    <origin xyz="0 -3 0" rpy="0 0 1.5708"/>
-    <parent link="base_link"/>
-    <child link="side_camera_base"/>
-  </joint>-->
-  <!-- Camera -->
-  <!--<link name="side_camera_base">-->
-    <!-- <collision>
-      <origin xyz="0 0 0" rpy="0 0 0"/>
-      <geometry>
-        <box size="0.05 0.05 0.05"/>
-      </geometry>
-    </collision>
-    <visual>
-      <origin xyz="0 0 0" rpy="0 0 0"/>
-      <geometry>
-        <box size="0.05 0.05 0.05"/>
-      </geometry>
-      <material name="red"/>
-    </visual>
-    -->
-    <!--<inertial>
-      <mass value="1e-5" />
-      <origin xyz="0 0 0" rpy="0 0 0"/>
-      <inertia ixx="1e-6" ixy="0" ixz="0" iyy="1e-6" iyz="0" izz="1e-6" />
-    </inertial>
-  </link>-->
-  <!--
-  <link name="odom">
-    <collision>
-      <origin xyz="0 0 0" rpy="0 0 0"/>
-      <geometry>
-        <box size="0.1 0.1 0.1"/>
-      </geometry>
-  </collision>
-    </link>
-  <joint name="odom_joint" type="fixed">
-    <axis xyz="0 0 0" />
-    <origin xyz="0 0 0" rpy="0 0 0"/>
-    <parent link="odom"/>
-    <child link="base_link"/>
-  </joint>-->
-  <!--
-  <link name="lidar">
-    <xacro:null_inertial/>
-  </link>
-  <joint name="lidar_joint" type="fixed">
-    <origin xyz="0 0 0.1" rpy="0 0 0"/>
-    <parent link="chassis"/>
-    <child link="lidar"/>
-  </joint>
--->
   <!-- Wheels -->
   <xacro:front_wheel lr_prefix="left" fr_prefix="front"

Commit message: Fixed the geometry: - Better sizing - Wheels are now cylinders

File: urdf/traethlin.gazebo.xacro (robot description, xacro)
@@ -26,10 +26,14 @@
       <plugin name="depth_camera" filename="libgazebo_ros_camera.so">
         <ros>
-          <remapping>/camera/image_raw:=/camera/rgb/image_raw</remapping>
-          <remapping>/camera/image_raw/compressed:=/camera/rgb/image_raw/compressed</remapping>
-          <remapping>/camera/image_raw/compressedDepth:=/camera/rgb/image_raw/compressedDepth</remapping>
-          <remapping>/camera/image_raw/theora:=/camera/rgb/image_raw/theora</remapping>
-          <remapping>/camera/camera_info:=/camera/rgb/camera_info</remapping>
+          <remapping>/camera/image_raw:=/camera/color/image_raw</remapping>
+          <remapping>/camera/image_raw/compressed:=/camera/color/image_raw/compressed</remapping>
+          <remapping>/camera/image_raw/compressedDepth:=/camera/color/image_raw/compressedDepth</remapping>
+          <remapping>/camera/image_raw/theora:=/camera/color/image_raw/theora</remapping>
+          <remapping>/camera/camera_info:=/camera/color/camera_info</remapping>
           <remapping>/camera/points:=/camera/depth/points</remapping>
+          <remapping>/camera/depth/image_raw:=/camera/depth/image_rect_raw</remapping>
+          <remapping>/camera/depth/image_raw/compressed:=/camera/depth/image_rect_raw/compressed</remapping>
+          <remapping>/camera/depth/image_raw/compressedDepth:=/camera/depth/image_rect_raw/compressedDepth</remapping>
+          <remapping>/camera/depth/image_raw/theora:=/camera/depth/image_rect_raw/theora</remapping>
         </ros>
         <camera_name>camera</camera_name>
@@ -76,5 +80,5 @@
     <sensor name="imu" type="imu">
       <always_on>true</always_on>
-      <update_rate>10</update_rate>
+      <update_rate>100</update_rate>
       <imu>
         <angular_velocity>

File: urdf/traethlin.urdf.xacro (robot description, xacro)
@@ -133,5 +133,5 @@
       <origin xyz="0 0 0" rpy="0 0 0"/>
       <geometry>
-        <box size="0.15 0.15 0.07"/>
+        <box size="0.16 0.16 0.06"/>
       </geometry>
       <material name="lightgrey"/>
@@ -140,5 +140,5 @@
       <origin xyz="0 0 0" rpy="0 0 0"/>
       <geometry>
-        <box size="0.15 0.15 0.07"/>
+        <box size="0.16 0.16 0.06"/>
       </geometry>
     </collision>
@@ -146,5 +146,5 @@
   </link>
   <joint name="box_of_goodies_to_chassis_joint" type="fixed">
-    <origin xyz="-0.10 0 0.10" rpy="0 0 0"/>
+    <origin xyz="-0.108 0 0.115" rpy="0 0 0"/>
     <parent link="chassis_link"/>
     <child link="box_of_goodies_link"/>
@@ -175,5 +175,5 @@
   </link>
   <joint name="gps_joint" type="fixed">
-    <origin xyz="-0.10 0.0 0.14" rpy="0 0 0"/>
+    <origin xyz="-0.108 0.0 0.15" rpy="0 0 0"/>
     <parent link="chassis_link"/>
     <child link="gps_link"/>
@@ -199,10 +199,10 @@
   </gazebo>
   <joint name="cam_mount_joint" type="fixed">
-    <origin xyz="-0.19 0 0.04" rpy="0 0 0"/>
+    <origin xyz="-0.206 0 0.04" rpy="0 0 0"/>
     <parent link="chassis_link"/>
     <child link="cam_mount_link"/>
   </joint>
   <joint name="camera_base_joint" type="fixed">
-    <origin xyz="0.035 0 0.37" rpy="0 0.36 0"/>
+    <origin xyz="0.035 0 0.355" rpy="0 0.36 0"/>
     <parent link="cam_mount_link"/>
     <child link="camera_base"/>

File: urdf/traethlin_constants.xacro (robot description, xacro)
@@ -46,5 +46,5 @@
   <xacro:property name="rear_wheel_mass" value="0.89"/>-->
   <xacro:property name="hub_dia" value="0.015"/>
-  <xacro:property name="tire_dia" value="0.125"/>
+  <xacro:property name="tire_dia" value="0.110"/>
   <!-- <xacro:property name="hex_hub_depth" value="0.0"/>  -->
   <xacro:property name="front_tire_width" value="0.07"/>
@@ -59,7 +59,7 @@
   <xacro:property name="hex_hub_dist" value="0.4"/>-->
   <!-- The sum of the two wheelbases, front and rear, is the actual wheelbase  -->
-  <xacro:property name="wheelbase_front" value="0.312"/>
-  <xacro:property name="wheelbase_rear" value="0.312"/>
-  <xacro:property name="hex_hub_dist" value="0.22"/>
+  <xacro:property name="wheelbase_front" value="0.155"/>
+  <xacro:property name="wheelbase_rear" value="0.155"/>
+  <xacro:property name="hex_hub_dist" value="0.24"/>
   <!-- <xacro:property name="axle_length" value="0.03"/> -->
   <!--<xacro:property name="wheel_travel" value="0.1"/>

File: urdf/traethlin_shock_absorbers.xacro (robot description, xacro)
@@ -21,5 +21,5 @@
       ${-chassis_cm_height + front_shock_z_offset/2}"/>-->
       <origin xyz="${fr_reflect * chassis_cm_to_front_shock}
-                   ${lr_reflect * ((hex_hub_dist / 2) - 0.01)}
+                   ${lr_reflect * ((hex_hub_dist / 2) - 0.005)}
                    ${-front_shock_z_offset}"/>
       <axis xyz="0 0 -1"/>
@@ -47,10 +47,10 @@
       <parent link="chassis_link"/>
       <child link="${child}"/>
-      <!-- ${lr_reflect * ((hex_hub_dist / 2) + lr_reflect*(front_tire_width / 2))} -->
+      <!-- ${lr_reflect * ((hex_hub_dist / 2) + lr_reflect*(tire_width / 2))} -->
       <!--<origin xyz="${fr_reflect * chassis_cm_to_rear_shock}
                    ${lr_reflect * ((hex_hub_dist / 2) )}
       ${-chassis_height/2 + rear_shock_z_offset/2}"/>-->
       <origin xyz="${fr_reflect * chassis_cm_to_rear_shock}
-                   ${lr_reflect * ((hex_hub_dist / 2) - 0.01)}
+                   ${lr_reflect * ((hex_hub_dist / 2) - 0.005)}
                    ${-rear_shock_z_offset}"/>>
         <!-- rpy="0 0 ${lr_reflect*degrees_180}"/> -->

File: urdf/traethlin_wheels.xacro (robot description, xacro)
@@ -57,23 +57,18 @@
       <visual>
         <origin xyz="0 0 0" rpy="0 0 0"/>
+<!--
         <geometry>
           <mesh filename="${wheel_model}" scale="0.001 0.001 0.001"/>
         </geometry>
-        <!-- <geometry>
-          <cylinder radius="${tire_dia/2}" length="${rear_tire_width*0.1}"/>
-        </geometry> -->
+-->
+        <geometry>
+          <cylinder radius="${tire_dia/2}" length="${tire_width}"/>
+        </geometry>
         <material name="black"/>
       </visual>
-      <!--<collision name="collision">
-        <origin xyz="0 0 0" rpy="${degrees_90} 0 0"/>
-        <geometry>
-          <mesh filename="${wheel_model}" scale="0.632 0.632 0.661"/>
-        </geometry>
-      </collision>-->
       <collision name="collision">
         <origin xyz="0 0 0" rpy="0 0 0"/>
         <geometry>
-          <cylinder radius="${tire_dia/2}" length="${rear_tire_width*0.1}"/>
-          <!-- <mesh filename="${wheel_model}" scale="1 1 1"/> -->
+          <cylinder radius="${tire_dia/2}" length="${tire_width}"/>
         </geometry>
       </collision>

Commit message: Remapping of topics dependent on camera used.

File: urdf/traethlin.gazebo.xacro (robot description, xacro)
@@ -26,14 +26,31 @@
       <plugin name="depth_camera" filename="libgazebo_ros_camera.so">
         <ros>
-          <remapping>/camera/image_raw:=/camera/color/image_raw</remapping>
-          <remapping>/camera/image_raw/compressed:=/camera/color/image_raw/compressed</remapping>
-          <remapping>/camera/image_raw/compressedDepth:=/camera/color/image_raw/compressedDepth</remapping>
-          <remapping>/camera/image_raw/theora:=/camera/color/image_raw/theora</remapping>
-          <remapping>/camera/camera_info:=/camera/color/camera_info</remapping>
-          <remapping>/camera/points:=/camera/depth/points</remapping>
-          <remapping>/camera/depth/image_raw:=/camera/depth/image_rect_raw</remapping>
-          <remapping>/camera/depth/image_raw/compressed:=/camera/depth/image_rect_raw/compressed</remapping>
-          <remapping>/camera/depth/image_raw/compressedDepth:=/camera/depth/image_rect_raw/compressedDepth</remapping>
-          <remapping>/camera/depth/image_raw/theora:=/camera/depth/image_rect_raw/theora</remapping>
+          <xacro:property name="cmp_camera_type" value="$(arg camera_type)"/>
+          <!-- realsense d455 camera -->
+          <xacro:if value="${cmp_camera_type == 'd455'}">
+            <remapping>/camera/image_raw:=/camera/color/image_raw</remapping>
+            <remapping>/camera/image_raw/compressed:=/camera/color/image_raw/compressed</remapping>
+            <remapping>/camera/image_raw/compressedDepth:=/camera/color/image_raw/compressedDepth</remapping>
+            <remapping>/camera/image_raw/theora:=/camera/color/image_raw/theora</remapping>
+            <remapping>/camera/camera_info:=/camera/color/camera_info</remapping>
+            <remapping>/camera/points:=/camera/depth/points</remapping>
+            <remapping>/camera/depth/image_raw:=/camera/depth/image_rect_raw</remapping>
+            <remapping>/camera/depth/image_raw/compressed:=/camera/depth/image_rect_raw/compressed</remapping>
+            <remapping>/camera/depth/image_raw/compressedDepth:=/camera/depth/image_rect_raw/compressedDepth</remapping>
+            <remapping>/camera/depth/image_raw/theora:=/camera/depth/image_rect_raw/theora</remapping>
+          </xacro:if>
+          <!-- oak-d camera -->
+          <xacro:if value="${cmp_camera_type == 'oak-d-s2'}">
+            <remapping>camera/image_raw:=oak/rgb/image_raw</remapping>
+            <remapping>camera/image_raw/compressed:=oak/rgb/image_raw/compressed</remapping>
+            <remapping>camera/image_raw/compressedDepth:=oak/rgb/image_raw/compressedDepth</remapping>
+            <remapping>camera/image_raw/theora:=oak/rgb/image_raw/theora</remapping>
+            <remapping>camera/camera_info:=oak/rgb/camera_info</remapping>
+            <remapping>camera/points:=oak/points</remapping>
+            <remapping>camera/depth/image_raw:=oak/stereo/image_raw</remapping>
+            <remapping>camera/depth/image_raw/compressed:=oak/stereo/image_raw/compressed</remapping>
+            <remapping>camera/depth/image_raw/compressedDepth:=oak/stereo/image_raw/compressedDepth</remapping>
+            <remapping>camera/depth/image_raw/theora:=oak/stereo/image_raw/theora</remapping>
+          </xacro:if>
         </ros>
         <camera_name>camera</camera_name>

Commit message: Tweaked the urdf.

File: urdf/traethlin.gazebo.xacro (robot description, xacro)
@@ -14,14 +14,12 @@
     <sensor type="depth" name="camera">
       <update_rate>6.0</update_rate>
-      <!--<camera name="gazebo_camera">
-        <distortion>
-          <k1>0.1</k1>
-          <k2>0.2</k2>
-          <k3>0.3</k3>
-          <p1>0.4</p1>
-          <p2>0.5</p2>
-          <center>0.5 0.5</center>
-        </distortion>
-      </camera>-->
+      <camera name="camera">
+        <horizontal_fov>1.25664</horizontal_fov>
+        <!--<vertical_fov>0.855211</vertical_fov>-->
+        <image>
+          <width>320</width>
+          <height>180</height>
+        </image>
+      </camera>
       <plugin name="depth_camera" filename="libgazebo_ros_camera.so">
         <ros>
@@ -59,5 +57,5 @@
         <min_depth>0.04</min_depth>
         <max_depth>10.0</max_depth>
-        <hfov>87</hfov>
+        <!--<hfov>87</hfov>-->
       </plugin>
     </sensor>

File: urdf/traethlin.urdf.xacro (robot description, xacro)
@@ -128,5 +128,5 @@
   </link>
   <joint name="box_of_goodies_to_chassis_joint" type="fixed">
-    <origin xyz="-0.108 0 0.115" rpy="0 0 0"/>
+    <origin xyz="-0.105 0 0.115" rpy="0 0 0"/>
     <parent link="chassis_link"/>
     <child link="box_of_goodies_link"/>
@@ -181,5 +181,5 @@
   </gazebo>
   <joint name="cam_mount_joint" type="fixed">
-    <origin xyz="-0.206 0 0.04" rpy="0 0 0"/>
+    <origin xyz="-0.206 0 0.025" rpy="0 0 0"/>
     <parent link="chassis_link"/>
     <child link="cam_mount_link"/>
@@ -199,5 +199,5 @@
     </xacro:sensor_d455>
     <joint name="camera_base_joint" type="fixed">
-      <origin xyz="0.03 0 0.358" rpy="0 0.36 0"/>
+      <origin xyz="0.05 0 0.39" rpy="0 0.36 0"/>
       <parent link="cam_mount_link"/>
       <child link="camera_base"/>

File: urdf/traethlin_constants.xacro (robot description, xacro)
@@ -31,5 +31,5 @@
   <xacro:property name="chassis_vertical_offset" value="0.04"/>
   <xacro:property name="chassis_mass" value="1.5"/> <!-- excluding batteries-->
-  <xacro:property name="chassis_cm_height" value="0.10"/>
+  <xacro:property name="chassis_cm_height" value="0.09"/>
   <xacro:property name="chassis_cm_to_rear_shock" value="0.155"/>
   <xacro:property name="chassis_cm_to_front_shock" value="0.155"/>
