Commit message: First commit of the ignition branch

File: urdf/traethlin.gazebo.xacro (robot description, xacro)
@@ -12,6 +12,7 @@
 <robot name="traethlin" xmlns:xacro="http://www.ros.org/wiki/xacro">
   <gazebo reference="camera_base">
-    <sensor type="depth" name="camera">
+    <sensor type="rgbd_camera" name="camera">
       <update_rate>6.0</update_rate>
+      <topic>camera</topic>
       <camera name="camera">
         <horizontal_fov>1.25664</horizontal_fov>
@@ -22,5 +23,6 @@
         </image>
       </camera>
-      <plugin name="depth_camera" filename="libgazebo_ros_camera.so">
+      <gz_frame_id>camera_base</gz_frame_id>
+      <!--      <plugin name="depth_camera" filename="libgazebo_ros_camera.so">-->
         <ros>
           <xacro:property name="cmp_camera_type" value="$(arg camera_type)"/>
@@ -58,13 +60,14 @@
         <max_depth>10.0</max_depth>
         <!--<hfov>87</hfov>-->
-      </plugin>
+        <!--</plugin>-->
     </sensor>
   </gazebo>
   <gazebo reference="gps_link">
-    <material>Gazebo/Black</material>
-    <sensor name="gps" type="gps">
+    <material><xacro:gazebo_black/></material>
+    <sensor name="navsat" type="navsat">
+      <gz_frame_id>gps_link</gz_frame_id>
       <always_on>true</always_on>
       <update_rate>5</update_rate>
-      <gps>
+      <navsat>
         <position_sensing>
           <horizontal>
@@ -81,123 +84,41 @@
           </vertical>
         </position_sensing>
-      </gps>
-      <plugin name="gps_plugin" filename="libgazebo_ros_gps_sensor.so">
-        <ros>
-          <!-- <namespace>/traethlin</namespace> -->
-          <remapping>~/out:=gps/fix</remapping>
-          <remapping>~/vel:=gps/vel</remapping>
-          <frame_name>imu_link</frame_name>
-        </ros>
-      </plugin>
+      </navsat>
     </sensor>
   </gazebo>
   <gazebo reference="imu_link">
-    <sensor name="imu" type="imu">
-      <always_on>true</always_on>
-      <update_rate>100</update_rate>
-      <imu>
-        <angular_velocity>
-          <x>
-            <noise type="gaussian">
-              <mean>0.0</mean>
-              <stddev>2e-4</stddev>
-            </noise>
-          </x>
-          <y>
-            <noise type="gaussian">
-              <mean>0.0</mean>
-              <stddev>2e-4</stddev>
-            </noise>
-          </y>
-          <z>
-            <noise type="gaussian">
-              <mean>0.0</mean>
-              <stddev>2e-4</stddev>
-            </noise>
-          </z>
-        </angular_velocity>
-        <linear_acceleration>
-          <x>
-            <noise type="gaussian">
-              <mean>0.0</mean>
-              <stddev>1.7e-2</stddev>
-            </noise>
-          </x>
-          <y>
-            <noise type="gaussian">
-              <mean>0.0</mean>
-              <stddev>1.7e-2</stddev>
-            </noise>
-          </y>
-          <z>
-            <noise type="gaussian">
-              <mean>0.0</mean>
-              <stddev>1.7e-2</stddev>
-            </noise>
-          </z>
-        </linear_acceleration>
-      </imu>
-      <initial_orientation_as_reference>false</initial_orientation_as_reference>
-      <plugin name="imu" filename="libgazebo_ros_imu_sensor.so">
-        <ros>
-          <!-- <namespace>/traethlin</namespace> -->
-          <remapping>~/out:=imu/data</remapping>
-          <frame_name>imu_link</frame_name>
-        </ros>
-      </plugin>
+    <sensor name="imu_sensor" type="imu">
+      <always_on>1</always_on>
+      <update_rate>1</update_rate>
+      <visualize>true</visualize>
+      <topic>imu</topic>
+      <gz_frame_id>imu_link</gz_frame_id>
     </sensor>
   </gazebo>
   <gazebo reference="thermal_link">
-    <material>Gazebo/White</material>
-    <sensor type="camera" name="thermal_camera">
+    <material><xacro:gazebo_white/></material>
+    <sensor type="thermal" name="thermal_camera">
+      <topic>thermal_camera/image</topic>
       <camera name="thermal_camera">
         <horizontal_fov>1.92</horizontal_fov>
+        <!--
         <vertical_fov>1.31</vertical_fov>
+        -->
         <image>
           <width>16</width>
           <height>12</height>
+          <format>L8</format>
         </image>
       </camera>
-      <plugin name="thermal_camera" filename="libgazebo_ros_camera.so">
-        <ros>
-          <!-- <namespace>traethlin</namespace> -->
-<!--          <remapping>~/image_raw:=thermal_image</remapping>
-          <remapping>~/camera_info:=thermal_info</remapping>
-          -->
-          </ros>
-        <frame_name>thermal_link</frame_name>
-        <hack_baseline>0.07</hack_baseline>
+      <visualize>true</visualize>
+      <plugin
+          filename="ignition-gazebo-thermal-sensor-system"
+          name="gz::sim::systems::ThermalSensor">
+        <min_temp>200.0</min_temp>
+        <max_temp>300.0</max_temp>
+        <resolution>10</resolution>
       </plugin>
+      <frame_name>thermal_link</frame_name>
     </sensor>
   </gazebo>
-  <!--
-  <gazebo reference="lidar">
-    <sensor name="sensor_ray" type="ray">
-      <pose>0.5 0 0 0 0 0</pose>
-      <ray>
-        <scan>
-          <horizontal>
-            <samples>200</samples>
-            <resolution>1.0</resolution>
-            <min_angle>-0.74</min_angle>
-            <max_angle>0.74</max_angle>
-          </horizontal>
-        </scan>
-        <range>
-          <min>0.04</min>
-          <max>10.0</max>
-        </range>
-      </ray>
-      <always_on>true</always_on>
-      <visualize>true</visualize>
-      <update_rate>100.0</update_rate>
-      <plugin name="laser" filename="libgazebo_ros_ray_sensor.so">
-        <ros>
-          <remapping>laser/out:=laser_scan</remapping>
-        </ros>
-        <output_type>sensor_msgs/LaserScan</output_type>
-      </plugin>
-    </sensor>
-  </gazebo>
-  -->
 </robot>

File: urdf/traethlin.urdf.xacro (robot description, xacro)
@@ -13,8 +13,4 @@
   <xacro:arg name="camera_type" default="oak-d-s2" />
   <!-- Possible values are 'oak-d-s2' or 'd455' -->
-  <xacro:include filename="$(find traethlin_description)/urdf/traethlin_constants.xacro" />
-  <xacro:include filename="$(find traethlin_description)/urdf/traethlin_shock_absorbers.xacro" />
-  <xacro:include filename="$(find traethlin_description)/urdf/traethlin_wheels.xacro" />
-  <xacro:include filename="$(find traethlin_description)/urdf/traethlin.gazebo.xacro" />
   <material name="black">
     <color rgba="0.0 0.0 0.0 1"/>
@@ -32,4 +28,21 @@
     <color rgba="0.9 0.9 0.5 1"/>
   </material>
+  <!-- Gazebo colours -->
+  <!-- These are to be used inside a <material> tag in a <agzebo> tag. -->
+  <xacro:macro name="gazebo_black">
+    <ambient>0.0 0.0 0.0 1</ambient>
+    <diffuse>0.0 0.0 0.0 1</diffuse>
+    <specular>0.0 0.0 0.0 1</specular>
+  </xacro:macro>
+  <xacro:macro name="gazebo_white">
+    <ambient>1.0 1.0 1.0 1</ambient>
+    <diffuse>1.0 1.0 1.0 1</diffuse>
+    <specular>1.0 1.0 1.0 1</specular>
+  </xacro:macro>
+  <xacro:macro name="gazebo_grey">
+    <ambient>0.3 0.3 0.3 1</ambient>
+    <diffuse>0.7 0.7 0.7 1</diffuse>
+    <specular>0.01 0.01 0.01 1</specular>
+  </xacro:macro>
   <!-- Null inertial element. This is needed to make the model work with
        Gazebo. -->
@@ -55,5 +68,5 @@
         iyy="${(mass*(3*outer_rad*outer_rad+height*height))/12}"
         iyz = "0"
-        izz="${mass*outer_rad/2}"/>
+        izz="${mass*outer_rad*outer_rad/2}"/>
       <!-- izz above should have the outer_rad squared, but this makes the robot
       explode as soon as it moves. -->
@@ -71,8 +84,12 @@
     </inertial>
   </xacro:macro>
+  <xacro:include filename="$(find traethlin_description)/urdf/traethlin_constants.xacro" />
+  <xacro:include filename="$(find traethlin_description)/urdf/traethlin_shock_absorbers.xacro" />
+  <xacro:include filename="$(find traethlin_description)/urdf/traethlin_wheels.xacro" />
+  <xacro:include filename="$(find traethlin_description)/urdf/traethlin.gazebo.xacro" />
   <link name="base_link">
   </link>
   <gazebo reference="base_link">
-    <material>Gazebo/Grey</material>
+    <material><xacro:gazebo_grey/></material>
   </gazebo>
   <!-- Chassis -->
@@ -103,5 +120,9 @@
   </link>
   <gazebo reference="chassis_link">
-    <material>Gazebo/DarkGrey</material>
+    <material>
+      <ambient>0.175 0.175 0.175 1</ambient>
+      <diffuse>0.175 0.175 0.175 1</diffuse>
+      <specular>0.175 0.175 0.175 1</specular>
+    </material>
     <mu1>0.2</mu1>
     <mu2>0.2</mu2>
@@ -180,5 +201,9 @@
   </link>
   <gazebo reference="cam_mount_link">
-    <material>Gazebo/Orange</material>
+    <material>
+      <ambient>1.0 0.5 0.005 1</ambient>
+      <diffuse>1.0 0.5 0.005 1</diffuse>
+      <specular>1.0 0.5 0.005 1</specular>
+    </material>
   </gazebo>
   <joint name="cam_mount_joint" type="fixed">
@@ -270,42 +295,31 @@
                     axle_eff_limit="${rear_axle_eff_limit}"/>
   <gazebo>
-    <plugin name="gazebo_ros_ackermann_drive"
-            filename="libgazebo_ros_ackermann_drive_4wd.so">
-      <ros>
-        <!-- <namespace>traethlin</namespace> -->
-        <remapping>cmd_vel:=cmd_vel</remapping>
-        <remapping>odom:=odom</remapping>
-        <remapping>distance:=distance</remapping>
-      </ros>
-      <update_rate>100.0</update_rate>
-      <!-- wheels -->
-      <front_left_joint>left_front_axle</front_left_joint>
-      <front_right_joint>right_front_axle</front_right_joint>
-      <rear_left_joint>left_rear_axle</rear_left_joint>
-      <rear_right_joint>right_rear_axle</rear_right_joint>
+    <plugin
+      filename="gz-sim-ackermann-steering-system"
+      name="gz::sim::systems::AckermannSteering">
+      <left_joint>left_front_axle</left_joint>
+      <left_joint>left_rear_axle</left_joint>
+      <right_joint>right_front_axle</right_joint>
+      <right_joint>right_rear_axle</right_joint>
       <left_steering_joint>left_steering_joint</left_steering_joint>
       <right_steering_joint>right_steering_joint</right_steering_joint>
-      <steering_wheel_joint></steering_wheel_joint>
-      <!-- Max absolute steer angle for tyre in radians-->
-      <!-- Any cmd_vel angular z greater than this would be capped -->
-      <max_steer>0.7</max_steer>
-      <!-- Max absolute steering angle of steering wheel -->
-      <max_steering_angle>7.85</max_steering_angle>
-      <!-- Max absolute linear speed in m/s -->
-      <max_speed>1.5</max_speed>
-      <!-- PID tuning -->
-      <left_steering_pid_gain>100 20 1</left_steering_pid_gain>
-      <left_steering_i_range>0 0</left_steering_i_range>
-      <right_steering_pid_gain>100 20 1</right_steering_pid_gain>
-      <right_steering_i_range>0 0</right_steering_i_range>
-      <linear_velocity_pid_gain>5 1 0</linear_velocity_pid_gain>
-      <linear_velocity_i_range>0 0</linear_velocity_i_range>
-      <!-- output -->
-      <publish_odom>true</publish_odom>
-      <publish_odom_tf>true</publish_odom_tf>
-      <publish_wheel_tf>true</publish_wheel_tf>
-      <publish_distance>true</publish_distance>
-      <odometry_frame>odom</odometry_frame>
-      <robot_base_frame>base_link</robot_base_frame>
+      <kingpin_width>${hex_hub_dist}</kingpin_width>
+      <steering_limit>0.7</steering_limit>
+      <wheel_base>${wheelbase_front+wheelbase_rear}</wheel_base>
+      <wheel_separation>${hex_hub_dist}</wheel_separation>
+      <wheel_radius>${tyre_dia/2.0}</wheel_radius>
+      <min_velocity>-1</min_velocity>
+      <max_velocity>1.5</max_velocity>
+      <min_acceleration>-3</min_acceleration>
+      <max_acceleration>3</max_acceleration>
+      <odom_topic>odom</odom_topic>
+      <tf_topic>/tf</tf_topic>
+      <frame_id>odom</frame_id>
+      <child_frame_id>base_link</child_frame_id>
+    </plugin>
+    <plugin
+      filename="gz-sim-joint-state-publisher-system"
+      name="gz::sim::systems::JointStatePublisher">
+      <topic>joint_states</topic>
     </plugin>
   </gazebo>

File: urdf/traethlin_wheels.xacro (robot description, xacro)
@@ -78,5 +78,5 @@
     </link>
     <gazebo reference="${lr_prefix}_${fr_prefix}_wheel">
-      <material>Gazebo/Black</material>
+      <material><xacro:gazebo_black/></material>
       <mu1>10</mu1>
       <mu2>10</mu2>

Commit message: Added the possibility of using version 6 of gazebo, as well as the current (v8).

File: urdf/traethlin.gazebo.xacro (robot description, xacro)
@@ -113,11 +113,23 @@
       </camera>
       <visualize>true</visualize>
-      <plugin
-          filename="ignition-gazebo-thermal-sensor-system"
-          name="gz::sim::systems::ThermalSensor">
-        <min_temp>200.0</min_temp>
-        <max_temp>300.0</max_temp>
-        <resolution>10</resolution>
-      </plugin>
+      <xacro:property name="cmp_gazebo_major_version"
+                      value="$(arg gazebo_major_version)"/>
+      <xacro:if value="${cmp_gazebo_major_version == 8}">
+        <plugin filename="ignition-gazebo-thermal-sensor-system"
+                name="gz::sim::systems::ThermalSensor">
+          <min_temp>200.0</min_temp>
+          <max_temp>300.0</max_temp>
+          <resolution>10</resolution>
+        </plugin>
+      </xacro:if>
+      <xacro:if value="${cmp_gazebo_major_version == 6}">
+        <!-- For now we only have versions 6 and 8.  6 will disappear eventually-->
+        <plugin filename="ignition-gazebo-thermal-system"
+                name="gz::sim::systems::Thermal">
+          <min_temp>200.0</min_temp>
+          <max_temp>300.0</max_temp>
+          <resolution>10</resolution>
+        </plugin>
+      </xacro:if>
       <frame_name>thermal_link</frame_name>
     </sensor>

File: urdf/traethlin.urdf.xacro (robot description, xacro)
@@ -13,4 +13,5 @@
   <xacro:arg name="camera_type" default="oak-d-s2" />
   <!-- Possible values are 'oak-d-s2' or 'd455' -->
+  <xacro:arg name="gazebo_major_version" default="8" />
   <material name="black">
     <color rgba="0.0 0.0 0.0 1"/>
